Commit message: 5.8

File: src/urdftest/robot/robot.urdf (robot description, URDF)
Before this commit: robot myfirstrobot, 1 links, 0 joints
Links:
- removed link base_link
- added link link1
- added link link2
- added link link3
- added link link4
Joints:
- added joint joint1: type continuous, parent link1, child link2, origin xyz=5 3 0 rpy=0 0 0
- added joint joint2: type continuous, parent link1, child link3, origin xyz=-2 5 0 rpy=0 0 1.57
- added joint joint3: type continuous, parent link3, child link4, origin xyz=5 0 0 rpy=0 0 -1.57
